File: fan-controller.kicad_pcb (KiCad board)
At the start: 2 copper layers, 44.7 x 37.6 mm, 24 parts, among them J1 Conn_01x04_Pin, J2 Conn_01x04_Pin, J3 Conn_01x04_Pin, J4 12v, J5 Conn_01x04_Pin, Q1 Q_NMOS_GSD, Q2 Q_NMOS_GSD, Q3 Q_NMOS_GSD, U1 ESP32-S3-WROOM-1, U2 AMS1117-3.3

Commit message: Add backup files, Final layout
Parts:
- removed J4: 12v, Connector_BarrelJack:BarrelJack_Horizontal
- added C4: 22u, Capacitor_SMD:C_0805_2012Metric, F.Cu at (144.8, 81.0)
- added C5: 22u, Capacitor_SMD:C_0805_2012Metric, F.Cu at (141.1, 94.0)
- added D1: C7420331, Diode_SMD:D_SOD-323, F.Cu at (139.6, 90.2)
- added J6: USB_C_Receptacle_USB2.0_16P, Connector_USB:USB_C_Receptacle_HRO_TYPE-C-31-M-12, F.Cu at (151.7, 87.3)
- added L1: C2842153, Inductor_SMD:L_Chilisin_BMRB00050518-B, F.Cu at (143.3, 85.6)
- added R10: 5k1, Resistor_SMD:R_0402_1005Metric, F.Cu at (147.3, 79.2)
- added R11: 5k1, Resistor_SMD:R_0402_1005Metric, F.Cu at (146.3, 79.2)
- added R8: R, Resistor_SMD:R_0402_1005Metric, F.Cu at (140.1, 92.5)
- added R9: R, Resistor_SMD:R_0402_1005Metric, F.Cu at (142.1, 92.5)
- added U3: MT3608, Package_TO_SOT_SMD:SOT-23-6, F.Cu at (143.3, 90.2)
- Q1, Q2, Q3: footprint Package_TO_SOT_SMD:SOT-323_SC-70 -> Package_TO_SOT_SMD:SOT-523
- moved C1 12.6 mm to (145.7, 98.4)
- moved C2 12.6 mm to (145.7, 95.4)
- moved U2 12.1 mm to (150.9, 96.9)
Connections:
- C1 pad 1: +12V -> +5V
- U1 pad 13: unconnected-(U1-IO19-Pad13) -> USBD-
- U1 pad 14: unconnected-(U1-IO20-Pad14) -> USBD+
- U2 pad 3: +12V -> +5V
Routing:
- net USBD+: track 0.00 -> 32.4 mm, vias 0 -> 2
- net +5V: track 0.00 -> 31.9 mm
- net USBD-: track 0.00 -> 31.4 mm, vias 0 -> 2
- net Net-(J6-CC1): track 0.00 -> 13.9 mm
- net Net-(J6-CC2): track 0.00 -> 10.3 mm
- net +12V: track 55.1 -> 50.3 mm, vias 0 -> 2
- net GND: track 4.02 -> 8.52 mm, vias 24 -> 45
- net Net-(U3-FB): track 0.00 -> 2.56 mm
- net +3V3: track 48.9 -> 48.1 mm
- net Net-(J3-Pin_1): track 5.32 -> 5.83 mm
- net Net-(J2-Pin_1): track 5.42 -> 5.93 mm
Other:
- board text added: "EEAN"
